File: hardware/luftctl.kicad_sch (KiCad schematic)
At the start: 45 parts, among them J1 USB_C_Receptacle_USB2.0, J4 PWM Fan, J5 PWM Fan, J6 Conn_01x10, SW1 Reset, U3 USBLC6-4SC6, U4 ESP32-C3-WROOM-02, U5 CH224K, U6 LMR51420YFDDCR

Commit message: Compact layout: 56.7 x 32.1 mm, centred on fan headers and USB-C
- Outline centred on the fan headers (y 62.45); J1 moved down 5 mm to match.
- J6 along the bottom edge; buck and CH224K groups packed beside SW1 and
  under J1; D4/R16 above J1. TP1/TP4 removed.
- GND poured on both layers with via stitching; antenna keep-out extended.
- Re-routed; DRC 0 unconnected, no new violations; board matches schematic.
- CPL regenerated with JLCPCB rotation corrections; gerbers regenerated.

Co-Authored-By: Claude Opus 5.5 (1M context) <noreply@anthropic.com>
Parts:
- removed TP1, TP4: Test, TestPoint:TestPoint_THTPad_D1.5mm_Drill0.7mm, symbol Connector:TestPoint_Probe
Changed lines of the file:
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@@
-    (pin "1")
-  )
-  (symbol (lib_id "power:GND") (at 67.31 80.01 0) (unit 1)
-    (in_bom yes) (on_board yes)
-    (property "Reference" "#PWR0104" (id 0) (at 67.31 86.36 0)
-      (effects (font (size 1.27 1.27)) hide)
-    )
-    (property "Value" "GND" (id 1) (at 67.437 84.4042 0))
-    (property "Footprint" "" (id 2) (at 67.31 80.01 0)
-      (effects (font (size 1.27 1.27)) hide)
-    )
-    (property "Datasheet" "" (id 3) (at 67.31 80.01 0)
-      (effects (font (size 1.27 1.27)) hide)
-    )
     (pin "1")
   )
@@
     (pin "1")
     (pin "2")
-  )
-  (symbol (lib_id "Connector:TestPoint_Probe") (at 67.31 80.01 0) (unit 1)
-    (in_bom yes) (on_board yes) (fields_autoplaced)
-    (property "Reference" "TP4" (id 0) (at 71.12 77.1524 0)
-      (effects (font (size 1.27 1.27)) (justify left))
-    )
-    (property "Value" "Test" (id 1) (at 71.12 79.6924 0)
-      (effects (font (size 1.27 1.27)) (justify left))
-    )
-    (property "Footprint" "TestPoint:TestPoint_THTPad_D1.5mm_Drill0.7mm" (id 2) (at 72.39 80.01 0)
-      (effects (font (size 1.27 1.27)) hide)
-    )
-    (property "Datasheet" "~" (id 3) (at 72.39 80.01 0)
-      (effects (font (size 1.27 1.27)) hide)
-    )
-    (pin "1")
   )
   (symbol (lib_id "power:GND") (at 88.9 162.56 0) (unit 1)
@@
     (pin "4")
   )
-  (symbol (lib_id "Connector:TestPoint_Probe") (at 107.95 110.49 0) (unit 1)
-    (in_bom yes) (on_board yes) (fields_autoplaced)
-    (property "Reference" "TP1" (id 0) (at 111.76 107.6324 0)
-      (effects (font (size 1.27 1.27)) (justify left))
-    )
-    (property "Value" "Test" (id 1) (at 111.76 110.1724 0)
-      (effects (font (size 1.27 1.27)) (justify left))
-    )
-    (property "Footprint" "TestPoint:TestPoint_THTPad_D1.5mm_Drill0.7mm" (id 2) (at 113.03 110.49 0)
-      (effects (font (size 1.27 1.27)) hide)
-    )
-    (property "Datasheet" "~" (id 3) (at 113.03 110.49 0)
-      (effects (font (size 1.27 1.27)) hide)
-    )
-    (pin "1")
-  )
   (symbol (lib_id "Device:C_Small") (at 90.17 40.64 180) (unit 1)
     (in_bom yes) (on_board yes)
@@
       (reference "#PWR0103") (unit 1) (value "GND") (footprint "")
     )
-    (path "/9a9e9a4a-4d55-4aca-b958-cc420a7bca33"
-      (reference "#PWR0104") (unit 1) (value "GND") (footprint "")
-    )
     (path "/b74c8878-ebea-4c0e-af6a-e2125fba37ee"
       (reference "A1") (unit 1) (value "2022") (footprint "ansemjo:ahoi")
@@
       (reference "SW1") (unit 1) (value "Reset") (footprint "Button_Switch_SMD:SW_SPST_TS-1088-xR020")
     )
-    (path "/e2205131-398e-4b23-a7cb-6ed24a167152"
-      (reference "TP1") (unit 1) (value "Test") (footprint "TestPoint:TestPoint_THTPad_D1.5mm_Drill0.7mm")
-    )
     (path "/6d148275-a67a-4433-85c5-2078a8f76090"
       (reference "TP2") (unit 1) (value "Test") (footprint "TestPoint:TestPoint_THTPad_D1.5mm_Drill0.7mm")
@@
       (reference "TP3") (unit 1) (value "Test") (footprint "TestPoint:TestPoint_THTPad_D1.5mm_Drill0.7mm")
     )
-    (path "/a04199d5-1929-4c71-b1c1-ac84e1319139"
-      (reference "TP4") (unit 1) (value "Test") (footprint "TestPoint:TestPoint_THTPad_D1.5mm_Drill0.7mm")
-    )
     (path "/e7c5d7a0-c546-488a-8bb3-fe81c8ca39ca"

Commit message: Add J7/J8 switch headers (GPIO3, GPIO8) beside USB-C
- J7 (GPIO3+GND) above and J8 (GPIO8+GND) below the USB-C port on the
  right edge; ESPHome Switch 1/Switch 2 binary sensors with pull-ups.
- Remove R3 (old GPIO3 pull-down) so the switch input can idle high.
- J6 back to 8 pins (3V3, GND, IO2, RX, TX, GND, SDA, SCL).
- Tie CH224K CFG1/CFG2 directly to GND; drop R13/R14 0R straps.
- Edge no-track strips; FAN1_Tacho re-routed off the board edge.
- DRC 0 unconnected, no new errors; board matches schematic.

Co-Authored-By: Claude Opus 5.5 (1M context) <noreply@anthropic.com>
Parts:
- removed R13, R14: 0Ω, Resistor_SMD:R_0805_2012Metric_Pad1.20x1.40mm_HandSolder, symbol Device:R_Small
- removed R3: 10kΩ, Resistor_SMD:R_0805_2012Metric_Pad1.20x1.40mm_HandSolder, symbol Device:R_Small
- added J7: SW_IO3, Connector_PinHeader_2.54mm:PinHeader_1x02_P2.54mm_Vertical, symbol Connector_Generic:Conn_01x02
- added J8: SW_IO8, Connector_PinHeader_2.54mm:PinHeader_1x02_P2.54mm_Vertical, symbol Connector_Generic:Conn_01x02
- J6: value Conn_01x10 -> Conn_01x08; footprint Connector_PinHeader_2.54mm:PinHeader_1x10_P2.54mm_Vertical -> Connector_PinHeader_2.54mm:PinHeader_1x08_P2.54mm_Vertical; symbol Connector_Generic:Conn_01x10 -> Connector_Generic:Conn_01x08
Connections:
- net CFG1 is gone; now on net GND: U5.9 (CFG1)
- net CFG2 is gone; now on net GND: U5.2 (CFG2)
- net GND: now also J6.6 (Pin_6), J7.2 (Pin_2), J8.2 (Pin_2); no longer J6.8 (Pin_8)
- net GPIO3: now also J7.1 (Pin_1); no longer J6.4 (Pin_4)
- net GPIO8: now also J8.1 (Pin_1); no longer J6.5 (Pin_5)
- net RXD: now also J6.4 (Pin_4); no longer J6.6 (Pin_6)
- net SCL: now also J6.8 (Pin_8); no longer J6.10 (Pin_10)
- net SDA: now also J6.7 (Pin_7); no longer J6.9 (Pin_9)
- net TXD: now also J6.5 (Pin_5); no longer J6.7 (Pin_7)
